Commit message: Move world-base_link fixed link to top level xacro file

File: fanuc_lrmate200id_gazebo/urdf/lrmate200id.xacro (robot description, xacro)
@@ -4,3 +4,10 @@
   <xacro:include filename="$(find fanuc_lrmate200id_gazebo)/urdf/lrmate200id.gazebo"/>
   <xacro:fanuc_lrmate200id prefix=""/>
+  <!-- fix the base to the Gazebo world -->
+  <link name="world" />
+  <joint name="fixed" type="fixed">
+    <origin xyz="0 0 0" rpy="0 0 0"/>
+    <parent link="world"/>
+    <child link="base_link"/>
+  </joint>
 </robot>
